Commit message: fix typo & keyframe

File: tocabi_description/robots/dyros_tocabi_isaacsim.urdf (robot description, URDF)
Before this commit: robot dyros_tocabi_description, 62 links, 61 joints
Links:
- link act1_1: geometry collision mesh filename=package://tocabi_description/meshes/syhand/act1_1.stl scale=0.001 0.001 0.001; visual mesh filename=package://tocabi_description/meshes/syhand/act1_1.stl scale=0.001 0.001 0.001
- link act2_1: geometry collision mesh filename=package://tocabi_description/meshes/syhand/act2_1.stl scale=0.001 0.001 0.001; visual mesh filename=package://tocabi_description/meshes/syhand/act2_1.stl scale=0.001 0.001 0.001
- link act3_1: geometry collision mesh filename=package://tocabi_description/meshes/syhand/act3_1.stl scale=0.001 0.001 0.001; visual mesh filename=package://tocabi_description/meshes/syhand/act3_1.stl scale=0.001 0.001 0.001
- link act4_1: geometry collision mesh filename=package://tocabi_description/meshes/syhand/act4_1.stl scale=0.001 0.001 0.001; visual mesh filename=package://tocabi_description/meshes/syhand/act4_1.stl scale=0.001 0.001 0.001
- link dp1_1: geometry collision mesh filename=package://tocabi_description/meshes/syhand/dp1_1.stl scale=0.001 0.001 0.001; visual mesh filename=package://tocabi_description/meshes/syhand/dp1_1.stl scale=0.001 0.001 0.001
- link dp2_1: geometry collision mesh filename=package://tocabi_description/meshes/syhand/dp2_1.stl scale=0.001 0.001 0.001; visual mesh filename=package://tocabi_description/meshes/syhand/dp2_1.stl scale=0.001 0.001 0.001
- link dp3_1: geometry collision mesh filename=package://tocabi_description/meshes/syhand/dp3_1.stl scale=0.001 0.001 0.001; visual mesh filename=package://tocabi_description/meshes/syhand/dp3_1.stl scale=0.001 0.001 0.001
- link dp4_1: geometry collision mesh filename=package://tocabi_description/meshes/syhand/dp4_1.stl scale=0.001 0.001 0.001; visual mesh filename=package://tocabi_description/meshes/syhand/dp4_1.stl scale=0.001 0.001 0.001
- link mcp1_1: geometry collision mesh filename=package://tocabi_description/meshes/syhand/mcp1_1.stl scale=0.001 0.001 0.001; visual mesh filename=package://tocabi_description/meshes/syhand/mcp1_1.stl scale=0.001 0.001 0.001
- link mcp2_1: geometry collision mesh filename=package://tocabi_description/meshes/syhand/mcp2_1.stl scale=0.001 0.001 0.001; visual mesh filename=package://tocabi_description/meshes/syhand/mcp2_1.stl scale=0.001 0.001 0.001
- link mcp3_1: geometry collision mesh filename=package://tocabi_description/meshes/syhand/mcp3_1.stl scale=0.001 0.001 0.001; visual mesh filename=package://tocabi_description/meshes/syhand/mcp3_1.stl scale=0.001 0.001 0.001
- link mcp4_1: geometry collision mesh filename=package://tocabi_description/meshes/syhand/mcp4_1.stl scale=0.001 0.001 0.001; visual mesh filename=package://tocabi_description/meshes/syhand/mcp4_1.stl scale=0.001 0.001 0.001
- link meta1_1: geometry collision mesh filename=package://tocabi_description/meshes/syhand/meta1_1.stl scale=0.001 0.001 0.001; visual mesh filename=package://tocabi_description/meshes/syhand/meta1_1.stl scale=0.001 0.001 0.001
- link meta2_1: geometry collision mesh filename=package://tocabi_description/meshes/syhand/meta2_1.stl scale=0.001 0.001 0.001; visual mesh filename=package://tocabi_description/meshes/syhand/meta2_1.stl scale=0.001 0.001 0.001
- link meta3_1: geometry collision mesh filename=package://tocabi_description/meshes/syhand/meta3_1.stl scale=0.001 0.001 0.001; visual mesh filename=package://tocabi_description/meshes/syhand/meta3_1.stl scale=0.001 0.001 0.001
- link meta4_1: geometry collision mesh filename=package://tocabi_description/meshes/syhand/meta4_1.stl scale=0.001 0.001 0.001; visual mesh filename=package://tocabi_description/meshes/syhand/meta4_1.stl scale=0.001 0.001 0.001
- link mp1_1: geometry collision mesh filename=package://tocabi_description/meshes/syhand/mp1_1.stl scale=0.001 0.001 0.001; visual mesh filename=package://tocabi_description/meshes/syhand/mp1_1.stl scale=0.001 0.001 0.001
- link mp2_1: geometry collision mesh filename=package://tocabi_description/meshes/syhand/mp2_1.stl scale=0.001 0.001 0.001; visual mesh filename=package://tocabi_description/meshes/syhand/mp2_1.stl scale=0.001 0.001 0.001
- link mp3_1: geometry collision mesh filename=package://tocabi_description/meshes/syhand/mp3_1.stl scale=0.001 0.001 0.001; visual mesh filename=package://tocabi_description/meshes/syhand/mp3_1.stl scale=0.001 0.001 0.001
- link mp4_1: geometry collision mesh filename=package://tocabi_description/meshes/syhand/mp4_1.stl scale=0.001 0.001 0.001; visual mesh filename=package://tocabi_description/meshes/syhand/mp4_1.stl scale=0.001 0.001 0.001
- link palm: geometry collision mesh filename=package://tocabi_description/meshes/syhand/base_link.stl scale=0.001 0.001 0.001; visual mesh filename=package://tocabi_description/meshes/syhand/base_link.stl scale=0.001 0.001 0.001
- link pp1_1: geometry collision mesh filename=package://tocabi_description/meshes/syhand/pp1_1.stl scale=0.001 0.001 0.001; visual mesh filename=package://tocabi_description/meshes/syhand/pp1_1.stl scale=0.001 0.001 0.001
- link pp2_1: geometry collision mesh filename=package://tocabi_description/meshes/syhand/pp2_1.stl scale=0.001 0.001 0.001; visual mesh filename=package://tocabi_description/meshes/syhand/pp2_1.stl scale=0.001 0.001 0.001
- link pp3_1: geometry collision mesh filename=package://tocabi_description/meshes/syhand/pp3_1.stl scale=0.001 0.001 0.001; visual mesh filename=package://tocabi_description/meshes/syhand/pp3_1.stl scale=0.001 0.001 0.001
- link pp4_1: geometry collision mesh filename=package://tocabi_description/meshes/syhand/pp4_1.stl scale=0.001 0.001 0.001; visual mesh filename=package://tocabi_description/meshes/syhand/pp4_1.stl scale=0.001 0.001 0.001
